File: seal_project/seal_project.kicad_sch (KiCad schematic)
At the start: 5 parts, among them SW1 SW_SPST

Commit message: updated files
Parts:
- removed SW1: SW_SPST, symbol Switch:SW_SPST
- added SW1: SW_SPDT, Button_Switch_SMD:Nidec_Copal_CAS-120A, symbol Switch:SW_SPDT
- BT1: footprint (none) -> Battery:BatteryHolder_Keystone_106_1x20mm
Connections:
- net at D2.1 (K): now also R1.2; no longer D1.2 (A)
- net at D2.2 (A): now also D1.1 (K); no longer R1.1
- net at BT1.1 (+): now also SW1.1 (A)
- net at BT1.2 (-): now also D1.2 (A); no longer R1.2
- new net: R1.1, SW1.2 (B)
Other:
- moved on the sheet: D1, D2, R1
Changed lines of the file:
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@@
 (kicad_sch (version 20230121) (generator eeschema)
   (paper "A4")
-  (wire (pts (xy 124.46 86.36) (xy 138.43 86.36))
+  (wire (pts (xy 152.4 86.36) (xy 152.4 109.22))
     (stroke (width 0) (type default))
   )
@@
     (stroke (width 0) (type default))
   )
-  (wire (pts (xy 156.21 97.79) (xy 156.21 109.22))
+  (wire (pts (xy 152.4 109.22) (xy 132.08 109.22))
     (stroke (width 0) (type default))
   )
-  (wire (pts (xy 146.05 86.36) (xy 156.21 86.36))
-    (stroke (width 0) (type default))
-  )
-  (wire (pts (xy 156.21 109.22) (xy 132.08 109.22))
-    (stroke (width 0) (type default))
-  )
-  (wire (pts (xy 107.95 86.36) (xy 116.84 86.36))
-    (stroke (width 0) (type default))
-  )
-  (wire (pts (xy 107.95 92.71) (xy 107.95 86.36))
+  (wire (pts (xy 105.41 86.36) (xy 105.41 92.71))
     (stroke (width 0) (type default))
   )
@@
     (stroke (width 0) (type default))
   )
-  (wire (pts (xy 156.21 86.36) (xy 156.21 90.17))
+  (wire (pts (xy 105.41 86.36) (xy 107.95 86.36))
     (stroke (width 0) (type default))
   )
-  (symbol (lib_id "Device:LED") (at 142.24 86.36 0) (unit 1)
+  (wire (pts (xy 134.62 86.36) (xy 144.78 86.36))
+    (stroke (width 0) (type default))
+  )
+  (wire (pts (xy 115.57 86.36) (xy 127 86.36))
+    (stroke (width 0) (type default))
+  )
+  (symbol (lib_id "Device:LED") (at 130.81 86.36 0) (unit 1)
     (in_bom yes) (on_board yes) (dnp no) (fields_autoplaced)
-    (property "Reference" "D2" (at 140.6525 80.01 0)
+    (property "Reference" "D2" (at 129.2225 80.01 0)
       (effects (font (size 1.27 1.27)))
     )
-    (property "Value" "LED" (at 140.6525 82.55 0)
+    (property "Value" "LED" (at 129.2225 82.55 0)
       (effects (font (size 1.27 1.27)))
     )
-    (property "Footprint" "LED_THT:LED_D5.0mm" (at 142.24 86.36 0)
+    (property "Footprint" "LED_THT:LED_D5.0mm" (at 130.81 86.36 0)
       (effects (font (size 1.27 1.27)) hide)
     )
-    (property "Datasheet" "~" (at 142.24 86.36 0)
+    (property "Datasheet" "~" (at 130.81 86.36 0)
       (effects (font (size 1.27 1.27)) hide)
     )
@@
       (effects (font (size 1.27 1.27)))
     )
-    (property "Footprint" "" (at 128.016 109.22 90)
+    (property "Footprint" "Battery:BatteryHolder_Keystone_106_1x20mm" (at 128.016 109.22 90)
       (effects (font (size 1.27 1.27)) hide)
     )
@@
     )
   )
-  (symbol (lib_id "Device:LED") (at 120.65 86.36 0) (unit 1)
+  (symbol (lib_id "Switch:SW_SPDT") (at 105.41 97.79 270) (unit 1)
     (in_bom yes) (on_board yes) (dnp no) (fields_autoplaced)
-    (property "Reference" "D1" (at 119.0625 80.01 0)
+    (property "Reference" "SW1" (at 109.22 96.52 90)
+      (effects (font (size 1.27 1.27)) (justify left))
+    )
+    (property "Value" "SW_SPDT" (at 109.22 99.06 90)
+      (effects (font (size 1.27 1.27)) (justify left))
+    )
+    (property "Footprint" "Button_Switch_SMD:Nidec_Copal_CAS-120A" (at 105.41 97.79 0)
+      (effects (font (size 1.27 1.27)) hide)
+    )
+    (property "Datasheet" "~" (at 105.41 97.79 0)
+      (effects (font (size 1.27 1.27)) hide)
+    )
+    (pin "1")
+    (pin "2")
+    (pin "3")
+    (instances
+      (project "seal_project"
+        (path "/5ceb84d4-b9b1-477c-a057-6e0587106f91"
+          (reference "SW1") (unit 1)
+        )
+      )
+    )
+  )
+  (symbol (lib_id "Device:LED") (at 148.59 86.36 0) (unit 1)
+    (in_bom yes) (on_board yes) (dnp no) (fields_autoplaced)
+    (property "Reference" "D1" (at 147.0025 80.01 0)
       (effects (font (size 1.27 1.27)))
     )
-    (property "Value" "LED" (at 119.0625 82.55 0)
+    (property "Value" "LED" (at 147.0025 82.55 0)
       (effects (font (size 1.27 1.27)))
     )
-    (property "Footprint" "LED_THT:LED_D5.0mm" (at 120.65 86.36 0)
+    (property "Footprint" "LED_THT:LED_D5.0mm" (at 148.59 86.36 0)
       (effects (font (size 1.27 1.27)) hide)
     )
-    (property "Datasheet" "~" (at 120.65 86.36 0)
+    (property "Datasheet" "~" (at 148.59 86.36 0)
       (effects (font (size 1.27 1.27)) hide)
     )
@@
     )
   )
-  (symbol (lib_id "Switch:SW_SPST") (at 107.95 97.79 90) (unit 1)
+  (symbol (lib_id "Device:R") (at 111.76 86.36 90) (unit 1)
     (in_bom yes) (on_board yes) (dnp no) (fields_autoplaced)
-    (property "Reference" "SW1" (at 109.22 96.52 90)
-      (effects (font (size 1.27 1.27)) (justify right))
+    (property "Reference" "R1" (at 111.76 80.01 90)
+      (effects (font (size 1.27 1.27)))
     )
-    (property "Value" "SW_SPST" (at 109.22 99.06 90)
-      (effects (font (size 1.27 1.27)) (justify right))
+    (property "Value" "R" (at 111.76 82.55 90)
+      (effects (font (size 1.27 1.27)))
     )
-    (property "Footprint" "" (at 107.95 97.79 0)
+    (property "Footprint" "Resistor_THT:R_Axial_DIN0207_L6.3mm_D2.5mm_P7.62mm_Horizontal" (at 111.76 88.138 90)
       (effects (font (size 1.27 1.27)) hide)
     )
-    (property "Datasheet" "~" (at 107.95 97.79 0)
+    (property "Datasheet" "~" (at 111.76 86.36 0)
       (effects (font (size 1.27 1.27)) hide)
     )
-    (pin "1")
-    (pin "2")
-    (instances
-      (project "seal_project"
-        (path "/5ceb84d4-b9b1-477c-a057-6e0587106f91"
-          (reference "SW1") (unit 1)
-        )
-      )
-    )
-  )
-  (symbol (lib_id "Device:R") (at 156.21 93.98 0) (unit 1)
-    (in_bom yes) (on_board yes) (dnp no) (fields_autoplaced)
-    (property "Reference" "R1" (at 158.75 92.71 0)
-      (effects (font (size 1.27 1.27)) (justify left))
-    )
-    (property "Value" "R" (at 158.75 95.25 0)
-      (effects (font (size 1.27 1.27)) (justify left))
-    )
-    (property "Footprint" "Resistor_THT:R_Axial_DIN0207_L6.3mm_D2.5mm_P7.62mm_Horizontal" (at 154.432 93.98 90)
-      (effects (font (size 1.27 1.27)) hide)
-    )
-    (property "Datasheet" "~" (at 156.21 93.98 0)
-      (effects (font (size 1.27 1.27)) hide)
-    )

Commit message: Adds
Connections:
- net at D2.1 (K): now also D1.2 (A); no longer R1.2
- net at D2.2 (A): now also R1.2; no longer D1.1 (K)
- net at BT1.2 (-): now also D1.1 (K); no longer D1.2 (A)
Other:
- moved on the sheet: D1, D2

Commit message: updates, still debugging
Connections:
- net GND: now reaches SW1.3 (C)
Changed lines of the file:
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@@
+		)
+	)
+	(symbol
+		(lib_id "power:GND")
+		(at 102.87 102.87 0)
+		(unit 1)
+		(exclude_from_sim no)
+		(in_bom yes)
+		(on_board yes)
+		(dnp no)
+		(fields_autoplaced yes)
+		(property "Reference" "#PWR01"
+			(at 102.87 109.22 0)
+			(effects
+				(font
+					(size 1.27 1.27)
+				)
+				(hide yes)
+			)
+		)
+		(property "Value" "GND"
+			(at 102.87 107.95 0)
+			(effects
+				(font
+					(size 1.27 1.27)
+				)
+			)
+		)
+		(property "Footprint" ""
+			(at 102.87 102.87 0)
+			(effects
+				(font
+					(size 1.27 1.27)
+				)
+				(hide yes)
+			)
+		)
+		(property "Datasheet" ""
+			(at 102.87 102.87 0)
+			(effects
+				(font
+					(size 1.27 1.27)
+				)
+				(hide yes)
+			)
+		)
+		(property "Description" "Power symbol creates a global label with name \"GND\" , ground"
+			(at 102.87 102.87 0)
+			(effects
+				(font
+					(size 1.27 1.27)
+				)
+				(hide yes)
+			)
+		)
+		(pin "1"
+		)
+		(instances
+			(project ""
+				(path "/5ceb84d4-b9b1-477c-a057-6e0587106f91"
+					(reference "#PWR01")
+					(unit 1)
+				)
+			)
 		)
 	)
