File: seal_project/seal_project.kicad_pcb (KiCad board)
At the start: 2 copper layers, 72.1 x 63.5 mm, 6 parts, among them SW1 SW_SPDT

Commit message: done
Parts:
- removed G***: LOGO, LOGO
Other:
- board size 72.1 x 63.5 mm -> 74.8 x 67.4 mm

Commit message: ready to fab
Other:
- board text added: "|\__/,| (`\ _.|o o |_ ) ) -(((---(((-----"
Changed lines of the file:
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@@
 		(layer "Edge.Cuts")
+	)
+	(gr_text "    |\\__/,|  (`\\\n  _.|o o  |_  ) )\n-(((---(((-----"
+		(at 160.5 96 0)
+		(layer "B.SilkS")
+		(effects
+			(font
+				(size 1 1)
+				(thickness 0.15)
+			)
+			(justify left bottom)
+		)
 	)
 	(gr_text "To: Ezzat\nFrom: Cal"
